File: esp32s3_http.kicad_pcb (KiCad board)
At the start: 2 copper layers, 55 x 90 mm, 44 parts, among them J1 USB_B, J2 Jack-DC, J3 EXP1_UART, J4 EXP2, SW1 SW_Push, SW2 SW_Push, U1 ESP32-S3-WROOM-1, U2 LM2940T-3.3, U3 NJM7805FA, Y1 32.768KHz

Commit message: 回路図: 部品値を秋月の調達品に合わせる
- C8 47uF -> 22uF Ta, C4/C10 3.3uF -> 4.7uF, C9 3.3uF -> 1uF/25V
- C5/C6 12pF -> 15pF, R4 2.2k -> 1k

Co-Authored-By: Claude Opus 5.5 <noreply@anthropic.com>
Parts:
- C10, C4: value 3.3uF -> 4.7uF/10V
- C5, C6: value 12pF -> 15pF
- C8: value 47uF/10V Ta -> 22uF/10V Ta
- C9: value 3.3uF -> 1uF/25V
- R4: value 2.2k -> 1k
Changed lines of the file:
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@@
 			)
 		)
-		(property "Value" "3.3uF"
+		(property "Value" "1uF/25V"
 			(at 0 1.43 180)
 			(layer "F.Fab")
@@
 			)
 		)
-		(property "Value" "12pF"
+		(property "Value" "15pF"
 			(at 0 1.43 90)
 			(layer "F.Fab")
@@
 			)
 		)
-		(property "Value" "2.2k"
+		(property "Value" "1k"
 			(at 0 1.43 0)
 			(layer "F.Fab")
@@
 			)
 		)
-		(property "Value" "3.3uF"
+		(property "Value" "4.7uF/10V"
 			(at 0 1.43 180)
 			(layer "F.Fab")
@@
 			)
 		)
-		(property "Value" "3.3uF"
+		(property "Value" "4.7uF/10V"
 			(at 0 1.43 0)
 			(layer "F.Fab")
@@
 			)
 		)
-		(property "Value" "12pF"
+		(property "Value" "15pF"
 			(at 0 1.43 90)
 			(layer "F.Fab")
@@
 			)
 		)
-		(property "Value" "47uF/10V Ta"
+		(property "Value" "22uF/10V Ta"
 			(at 0 2.35 0)
 			(layer "F.Fab")

Commit message: SW1/SW2 と J2 を秋月品 (TS-06104 / MJ-179PH) 用フットプリントに変更
- プロジェクトローカルライブラリ esp32s3_http.pretty を追加 (${KIPRJMOD})
- SW_TS-06104: データシート P.C.B LAYOUT 準拠 (10.0/6.4 x 5.5/3.5)
- DCJack_MJ-179PH: スロット穴 3 本、部品面視 (データシートの穴図は半田面視)

Co-Authored-By: Claude Opus 5.5 <noreply@anthropic.com>
Parts:
- J2: value Jack-DC -> MJ-179PH; footprint Connector_BarrelJack:BarrelJack_GCT_DCJ200-10-A_Horizontal -> esp32s3_http:DCJack_MJ-179PH
- SW1, SW2: value SW_Push -> TS-06104; footprint Button_Switch_SMD:SW_Push_1P1T_NO_CK_KSC6xxJ -> esp32s3_http:SW_TS-06104
- moved J2 0.10 mm to (51.4, 130.0), turned to 0 degrees
Routing:
- net VDD33: track 196.7 -> 183.5 mm
- net BOOT: track 75.8 -> 82.3 mm
- net Net-(D4-A): track 9.19 -> 4.51 mm
- net 5V: track 125.4 -> 129.5 mm
- net Net-(D5-A): track 4.51 -> 8.34 mm
- net GPIO47: track 29.5 -> 26.6 mm
- net GPIO5: track 28.9 -> 26.3 mm
- net Net-(U1-IO15): track 12.6 -> 14.6 mm
- net EN: track 126.4 -> 127.9 mm
- net GPIO4: track 23.9 -> 23.0 mm
- net DM: track 43.0 -> 42.1 mm
- net GPIO7: track 27.0 -> 27.7 mm
- net GPIO6: track 26.4 -> 25.7 mm
- net DP: track 45.4 -> 46.0 mm

Commit message: J1 を秋月品 USB-B (5075BR-04) 用フットプリントに変更
- データシート PCB LAYOUT 準拠: 信号 2.50x2.00 d0.92, シェル 12.04 間隔 d2.30
- 旧 Lumberg 2411-02 からシェル穴位置が 0.15mm 異なる

Co-Authored-By: Claude Opus 5.5 <noreply@anthropic.com>
Parts:
- J1: value USB_B -> 5075BR-04; footprint Connector_USB:USB_B_Lumberg_2411_02_Horizontal -> esp32s3_http:USB_B_5075BR-04
- turned J1 to 0 degrees

Commit message: PCB: 基板の角を R3 に、シルクスクリーンを装飾
- 表: 縦書きタイトル (ESP32-S3 白抜き + HTTP)、RESET/BOOT ラベル
- 裏: 八角形タイトルパネル (ロゴ・仕様・rev・設計者)、Wi-Fi マーク (アンテナ方向)、
  端のコネクタ表示 LAN/USB/DC 7.5-12V とセンタープラス極性記号
- 装飾部はステッチングビアを除外、小文字はストロークフォント (0.15mm)

Co-Authored-By: Claude Opus 5.5 <noreply@anthropic.com>
Routing:
- net GND: vias 67 -> 47
Other:
- board text added: "ANT"
- board text added: "BOOT"
- board text added: "DC 7.5-12V"
- board text added: "ESP32-S3"
- board text added: "HTTP"
- board text added: "HTTP NODE"
- board text added: "RESET"
- board text added: "USB"
- board text added: "USB / DC 7.5-12V"
- board text added: "Wi-Fi + W5500 LAN"
- board text added: "design: sanbungi"
- board text added: "microSD / 13 GPIO"
- board text added: "rev 1.0 2026-10"

Commit message: シルク: ポテトサーバーのテーマでポテトを配置
- 表: ESP32 と W5500 の間にポテト (9mm アウトライン)、下の F.Cu は配線禁止にして迂回
- 裏: パネル副題を POTATO SERVER に、"powered by <ポテト>" バッジ、
  Wi-Fi マークの発信源をポテトに
- 画像: Fluent Emoji Potato (MIT, Microsoft) — art/ATTRIBUTION.md

Co-Authored-By: Claude Opus 5.5 <noreply@anthropic.com>
Routing:
- net W5500_CS: track 49.0 -> 32.9 mm, vias 1 -> 2
- net 5V: track 129.5 -> 115.3 mm
- net GPIO6: track 25.7 -> 30.3 mm
- net BOOT: track 82.3 -> 77.7 mm
- net Net-(D5-A): track 8.34 -> 4.51 mm
- net LED_STAT: track 45.6 -> 41.9 mm
- net VDD33: track 183.5 -> 180.4 mm
- net GPIO47: track 26.6 -> 29.6 mm
- net GPIO7: track 27.7 -> 27.0 mm
- net GND: vias 47 -> 40
Other:
- board text added: "POTATO SERVER"
- board text added: "powered by"
- board text removed: "HTTP NODE"
