File: esp32s3_http.kicad_pcb (KiCad board)
At the start: 2 copper layers, 55 x 90 mm, 44 parts, among them J1 5075BR-04, J2 MJ-179PH, J3 EXP1_UART, J4 EXP2, SW1 TS-06104, SW2 TS-06104, U1 ESP32-S3-WROOM-1, U2 LM2940T-3.3, U3 NJM7805FA, Y1 32.768KHz

Commit message: シルク: 表のタイトルを「ポテトでできた」おちゃめな文字に
- Chewy フォントを多角形化、1 文字ずつランダムな傾き・上下のゆらぎ
- 各文字にポテトの芽の小穴、ESP32 と HTTP の間に小さなポテト
- art/ATTRIBUTION.md に Chewy (Apache-2.0) を追記

Co-Authored-By: Claude Opus 5.5 <noreply@anthropic.com>
Other:
- board text removed: "HTTP"
